File: pcb/Silviaduino/Silviaduino.kicad_pcb (KiCad board)
At the start: 4 copper layers, 66 x 63.5 mm, 45 parts, among them J1 RTD1 Conn, J10 UEXT_Host, J11 ESP8266, J12 Conn_01x02, J2 RTD 2 Conn, J3 SSR1 Conn, J4 SSR2 Conn, J5 SSR3 Conn, J6 PSSR Conn, J7 PXDCR Conn, J8 Btn Conn, J9 Enc Conn, Q1 2N7002, Q2 2N7002, Q3 2N7002, Q4 BSS138, Q5 BSS138, U1 HT7550-1-SOT89, U2 HT7533-1-SOT89, U3 Teensy4.1, U4 PCF8591, U5 MAX31865xAP, U6 MAX31865xAP

Commit message: WIP
Parts:
- removed C5, C6: 10 uF, Capacitor_SMD:C_0402_1005Metric
- removed C7, C8: 0.1 uF, Capacitor_SMD:C_0402_1005Metric
- removed J11: ESP8266, Connector_PinSocket_2.54mm:PinSocket_2x04_P2.54mm_Vertical
- removed J6: PSSR Conn, Connector_PinHeader_2.54mm:PinHeader_1x04_P2.54mm_Vertical
- removed R10, R11, R8, R9: 10K, Resistor_SMD:R_0402_1005Metric
- removed R4, R5: 10M, Resistor_SMD:R_0402_1005Metric
- removed R6, R7: 400R, Resistor_SMD:R_0402_1005Metric
- removed U5, U6: MAX31865xAP, Package_SO:SSOP-20_5.3x7.2mm_P0.65mm
- added IC1: ADS1248IPWR, ads1248:SOP65P640X120-28N, F.Cu at (164.6, 64.3)
- added IC2: TTGO_MICRO_32, ttgo:TTGOMICRO32, F.Cu at (168.1, 112.5)
- added Q6: 2N7002, Package_TO_SOT_SMD:SOT-23, F.Cu at (173.0, 79.5)
- Q4, Q5: value BSS138 -> 2N7002
- U4: value PCF8591 -> ADS1015IDGS; footprint Package_SO:SOIC-16W_7.5x10.3mm_P1.27mm -> Package_SO:TSSOP-10_3x3mm_P0.5mm
- moved J10 63.1 mm to (154.9, 77.7)
- moved Q4 47.7 mm to (164.1, 79.5), turned to 0 degrees
- moved U4 42.0 mm to (166.4, 72.9)
- moved C3 41.7 mm to (159.0, 53.9)
- moved U1 41.7 mm to (164.1, 54.4)
- moved C2 41.4 mm to (170.7, 53.1)
- moved Q5 37.3 mm to (168.6, 79.5), turned to 0 degrees
- moved C9 30.7 mm to (163.3, 82.8), turned to 0 degrees
- moved J9 27.9 mm to (200.7, 60.5)
- moved J7 15.3 mm to (200.7, 74.7)
- moved J12 15.2 mm to (200.7, 53.3)
- moved J3 13.5 mm to (154.9, 92.2)
- moved J4 13.5 mm to (154.9, 99.8)
- moved J8 13.5 mm to (154.9, 115.1)
- moved J5 13.5 mm to (154.9, 107.4)
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Connections:
- J7 pad 2: PRES_AIN -> PXDCR_AIN
- Q4 pad 2: I2C_SDA -> SENSOR_I2C_SCL_3V3
- Q4 pad 3: I2C_SDA_5V -> SENSOR_I2C_SCL_5V
- Q5 pad 2: I2C_SCL -> SENSOR_I2C_SDA_3V3
- Q5 pad 3: I2C_SCL_5V -> SENSOR_I2C_SDA_5V
- U3 pad 10: UEXT_TXD -> Net-(U3-Pad10)
- U3 pad 11: Net-(U3-Pad11) -> ESP_RES
- U3 pad 12: UEXT_SSEL -> SENSOR_ADS1248_CS
- U3 pad 13: UEXT_MOSI -> SENSOR_MOSI
- U3 pad 14: UEXT_MISO -> SENSOR_MISO
- U3 pad 16: Net-(U3-Pad16) -> SENSOR_I2C_SCL_3V3
- U3 pad 17: Net-(U3-Pad17) -> SENSOR_I2C_SDA_3V3
- U3 pad 18: TEMP_SPI_MOSI -> ESP_MOSI
- U3 pad 19: TEMP_SPI_SCK -> ESP_SCK
- U3 pad 2: TEMP_SPI_CS0 -> ESP_CS
- U3 pad 20: TEMP_DRDY0 -> ESP_TX
- U3 pad 21: TEMP_DRDY1 -> ESP_RX
- U3 pad 25: ESP8266_RST -> TEENSY_GPIO4
- U3 pad 26: RX_FROM_ESP8266 -> TEENSY_GPIO3
- U3 pad 27: TX_TO_ESP8266 -> TEENSY_GPIO2
- U3 pad 28: ESP8266_CHPD -> SENSOR_EXT2_CS
- U3 pad 29: ESP8266_GPIO0 -> SENSOR_EXT1_CS
- U3 pad 3: TEMP_SPI_MISO -> ESP_MISO
- U3 pad 30: TEMP_SPI_CS1 -> Net-(U3-Pad30)
- U3 pad 31: ESP8266_GPIO2 -> Net-(U3-Pad31)
- U3 pad 32: PROP_SSR_EN -> ESP_GPIO0
- U3 pad 33: Net-(U3-Pad33) -> ESP_BUSY
- U3 pad 35: UEXT_SCK -> SENSOR_SCK
- U3 pad 36: Net-(U3-Pad36) -> SENSOR_ADS1248_START
- U3 pad 37: Net-(U3-Pad37) -> SENSOR_ADS1248_DRDY
- U3 pad 38: I2C_SCL -> TEENSY_GPIO1
- U3 pad 39: I2C_SDA -> TEENSY_GPIO0
- U3 pad 9: UEXT_RXD -> Net-(U3-Pad9)
- U4 pad 1: PRES_AIN -> Net-(U4-Pad1)
- U4 pad 10: I2C_SCL_5V -> SENSOR_I2C_SCL_5V
- U4 pad 2: GND -> SENSOR_ADC_RDY_5V
- U4 pad 4: GND -> PXCDR_AIN
- U4 pad 5: GND -> Net-(TP7-Pad1)
- U4 pad 6: GND -> Net-(TP8-Pad1)
- U4 pad 7: GND -> Net-(TP9-Pad1)
- U4 pad 8: GND -> +5V
- U4 pad 9: I2C_SDA_5V -> SENSOR_I2C_SDA_5V
Routing:
- net TEMP_DVDD: track 188.7 -> 0.00 mm, vias 4 -> 0
- net +5V: track 172.9 -> 0.00 mm, vias 1 -> 0
- net GND: track 111.6 -> 0.00 mm, vias 6 -> 0
- net PROP_SSR_EN: track 64.9 -> 0.00 mm, vias 1 -> 0
- net +9V: track 56.8 -> 0.00 mm
- net TEMP_DRDY0: track 55.1 -> 0.00 mm, vias 1 -> 0
- net TEMP_SPI_MOSI: track 52.2 -> 0.00 mm, vias 2 -> 0
- net UEXT_SSEL: track 52.2 -> 0.00 mm
- net TEMP_SPI_SCK: track 49.8 -> 0.00 mm, vias 2 -> 0
- net UEXT_RXD: track 49.5 -> 0.00 mm
- net UEXT_MOSI: track 46.1 -> 0.00 mm
- net UEXT_TXD: track 44.6 -> 0.00 mm
- net UEXT_SCL: track 44.5 -> 0.00 mm
- net TEMP_DRDY1: track 43.0 -> 0.00 mm, vias 1 -> 0
- net TEMP_SPI_CS1: track 42.5 -> 0.00 mm
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- removed copper zone on In1.Cu, net GND
Other:
- board size 66 x 63.5 mm -> 50.8 x 76.2 mm

Commit message: PCB work
Parts:
- removed IC1: ADS1248IPWR, ads1248:SOP65P640X120-28N
- removed IC2: TTGO_MICRO_32, ttgo:TTGOMICRO32
- removed Q4, Q5, Q6: 2N7002, Package_TO_SOT_SMD:SOT-23
- added C1: 100 nF, Capacitor_SMD:C_0402_1005Metric, F.Cu at (161.3, 54.4)
- added C10: 10 nF, Capacitor_SMD:C_0402_1005Metric, F.Cu at (170.4, 55.4)
- added C11: 10 nF, Capacitor_SMD:C_0402_1005Metric, F.Cu at (170.4, 48.0)
- added C12: 10 nF, Capacitor_SMD:C_0402_1005Metric, F.Cu at (167.6, 48.0)
- added C13: 100 nF, Capacitor_SMD:C_0402_1005Metric, F.Cu at (167.6, 45.7)
- added C14: 10 nF, Capacitor_SMD:C_0402_1005Metric, F.Cu at (167.6, 43.4)
- added C5: 10 nF, Capacitor_SMD:C_0402_1005Metric, F.Cu at (170.4, 50.8)
- added C6: 10 nF, Capacitor_SMD:C_0402_1005Metric, F.Cu at (170.4, 43.4)
- added C7: 100 nF, Capacitor_SMD:C_0402_1005Metric, F.Cu at (170.4, 53.1)
- added C8: 100 nF, Capacitor_SMD:C_0402_1005Metric, F.Cu at (170.4, 45.7)
- added J11: PSSR Conn, Connector_PinHeader_2.54mm:PinHeader_1x04_P2.54mm_Vertical, F.Cu at (177.0, 95.2)
- added J13: Micro_SD_Card, Connector_Card:microSD_HC_Hirose_DM3AT-SF-PEJM5, F.Cu at (155.7, 121.9)
- added J14: Conn_ARM_JTAG_SWD_10, Connector_PinHeader_1.27mm:PinHeader_2x05_P1.27mm_Vertical_SMD, F.Cu at (168.9, 127.0)
- added J6: Display Conn, Connector_PinHeader_2.54mm:PinHeader_1x07_P2.54mm_Vertical, F.Cu at (161.3, 71.1)
- added R10: 1K, Resistor_SMD:R_0402_1005Metric, F.Cu at (171.7, 51.8)
- added R11: 1K, Resistor_SMD:R_0402_1005Metric, F.Cu at (171.7, 44.5)
- added R12: 1K, Resistor_SMD:R_0402_1005Metric, F.Cu at (171.7, 54.4)
- added R13: 1K, Resistor_SMD:R_0402_1005Metric, F.Cu at (171.7, 46.7)
- added R14: 1K, Resistor_SMD:R_0402_1005Metric, F.Cu at (166.4, 47.0)
- added R15: 680R, Resistor_THT:R_Axial_DIN0204_L3.6mm_D1.6mm_P5.08mm_Horizontal, F.Cu at (163.1, 43.2)
- added R16: 1K, Resistor_SMD:R_0402_1005Metric, F.Cu at (166.4, 44.7)
- added R4: 4K7, Resistor_SMD:R_0402_1005Metric, F.Cu at (170.9, 61.5)
- added R5: 9K1, Resistor_SMD:R_0603_1608Metric, F.Cu at (170.9, 59.9)
- added R6: 9K1, Resistor_SMD:R_0603_1608Metric, F.Cu at (162.8, 94.5)
- added R7: 4K7, Resistor_SMD:R_0402_1005Metric, F.Cu at (161.8, 96.5)
- added R8: 3K6, Resistor_SMD:R_0603_1608Metric, F.Cu at (168.1, 104.1)
- added R9: 6K2, Resistor_SMD:R_0603_1608Metric, F.Cu at (169.9, 104.1)
- added U5: ADS1220xPW, Package_SO:TSSOP-16_4.4x5mm_P0.65mm, F.Cu at (165.6, 53.8)
- C2, C3, C4: footprint Capacitor_SMD:C_0402_1005Metric -> Capacitor_SMD:C_0603_1608Metric
- C9: value 0.1 uF -> 100 nF
- J1, J2: footprint Connector_PinHeader_2.54mm:PinHeader_1x04_P2.54mm_Vertical -> Connector_PinHeader_2.54mm:PinHeader_1x02_P2.54mm_Vertical
- U1: value HT7550-1-SOT89 -> 78S04; footprint Package_TO_SOT_SMD:SOT-89-3 -> Package_TO_SOT_THT:TO-220-3_Horizontal_TabDown
- U3: value Teensy4.1 -> MCP6002-xSN; footprint teensy:Teensy41 -> Package_SO:SOIC-8_3.9x4.9mm_P1.27mm
- U4: value ADS1015IDGS -> Portenta_H7; footprint Package_SO:TSSOP-10_3x3mm_P0.5mm -> Arduino:Arduino_Portenta_H7
- moved J12 99.6 mm to (133.1, 126.5)
- moved C2 76.0 mm to (133.1, 119.1), turned to 90 degrees
- moved C3 64.7 mm to (133.3, 113.3), turned to 270 degrees
- moved U1 60.3 mm to (144.0, 111.3), turned to 180 degrees
- moved J9 52.5 mm to (176.8, 107.2)
- moved J10 34.4 mm to (167.6, 109.7)
- moved J2 31.6 mm to (177.5, 51.8), turned to 0 degrees
- moved C9 30.5 mm to (161.3, 52.3), turned to 270 degrees
- moved J4 29.5 mm to (177.3, 80.5)
- moved J5 29.5 mm to (177.3, 88.1)
- moved J3 29.4 mm to (177.5, 73.4)
- moved J1 28.1 mm to (177.5, 44.5), turned to 0 degrees
- moved J7 27.8 mm to (177.5, 59.2)
- moved U3 26.9 mm to (166.9, 99.3), turned to 0 degrees
- moved Q1 24.5 mm to (171.5, 74.2), turned to 0 degrees
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Connections:
- net PXCDR_AIN renamed Net-(U4-Pad4)
- C2 pad 2: GND -> RTD2IN-
- C3 pad 2: GND -> RTD2IN-
- C4 pad 1: TEMP_VDD -> +3.3VA
- C4 pad 2: GND -> RTD2IN-
- C9 pad 1: TEMP_DVDD -> RTD2IN-
- C9 pad 2: GND -> +3V3
- D1 pad 1: GND -> RTD2IN-
- D2 pad 1: GND -> RTD2IN-
- D3 pad 1: GND -> RTD2IN-
- J1 pad 1: RTD1F- -> ADS1220_IDAC1_RTD1
- J1 pad 2: RTD1IN- -> ADS1220_IDAC1_RREF
- J10 pad 1: TEMP_DVDD -> +3V3
- J10 pad 10: UEXT_SSEL -> UEXT_CS
- J10 pad 2: GND -> RTD2IN-
- J10 pad 3: UEXT_TXD -> UART0_TX
- J10 pad 4: UEXT_RXD -> UART0_RX
- J10 pad 5: UEXT_SCL -> I2C0_SCL
- J10 pad 6: UEXT_SDA -> I2C0_SDA
- J10 pad 7: UEXT_MISO -> SPI5_MISO
- J10 pad 8: UEXT_MOSI -> SPI5_MOSI
- J10 pad 9: UEXT_SCK -> SPI5_SCK
- J12 pad 2: GND -> RTD2IN-
- J2 pad 1: RTD2F- -> RTD2IN-
- J2 pad 2: RTD2IN- -> ADS1220_IDAC1_RTD1
- J7 pad 1: GND -> RTD2IN-
- J8 pad 1: GND -> RTD2IN-
- J9 pad 4: TEMP_DVDD -> +3V3
- J9 pad 5: GND -> RTD2IN-
- Q1 pad 2: GND -> RTD2IN-
- Q2 pad 2: GND -> RTD2IN-
- Q3 pad 2: GND -> RTD2IN-
- U1 pad 1: GND -> +9V
- U1 pad 2: +9V -> RTD2IN-
- U2 pad 1: GND -> RTD2IN-
- U2 pad 2: +9V -> +5V
- U2 pad 3: TEMP_VDD -> +3.3VA
- U3 pad 1: GND -> PSSR_DAC_5V
- U3 pad 2: ESP_CS -> Net-(R6-Pad1)
- U3 pad 3: ESP_MISO -> PSSR_DAC_3V3
- U3 pad 4: SSR1_GATE -> RTD2IN-
- U3 pad 5: SSR2_GATE -> PSSR_EN_3V3
- U3 pad 6: SSR3_GATE -> Net-(R8-Pad1)
- U3 pad 7: Net-(U3-Pad7) -> PSSR_EN_9V
- U3 pad 8: Net-(U3-Pad8) -> +9V
- U4 pad 10: SENSOR_I2C_SCL_5V -> Net-(U4-Pad10)
- U4 pad 2: SENSOR_ADC_RDY_5V -> Net-(U4-Pad2)
- U4 pad 3: GND -> Net-(U4-Pad3)
- U4 pad 8: +5V -> Net-(U4-Pad8)
- U4 pad 9: SENSOR_I2C_SDA_5V -> Net-(U4-Pad9)
Routing:
- net RTD2IN-: track 0.00 -> 136.4 mm, vias 0 -> 24
- net Net-(R4-Pad2): track 0.00 -> 90.9 mm, vias 0 -> 2
- net JTAG_RESET: track 0.00 -> 90.0 mm, vias 0 -> 2
- net JTAG_TDO: track 0.00 -> 83.4 mm, vias 0 -> 2
- net JTAG_TCK: track 0.00 -> 82.6 mm, vias 0 -> 2
- net JTAG_TMS: track 0.00 -> 80.9 mm, vias 0 -> 2
- net ADS1220_DRDY: track 0.00 -> 76.3 mm, vias 0 -> 2
- net I2C0_SDA: track 0.00 -> 75.5 mm, vias 0 -> 1
- net ADS1220_CS: track 0.00 -> 75.3 mm, vias 0 -> 2
- net I2C0_SCL: track 0.00 -> 75.3 mm, vias 0 -> 1
- net SPI1_MOSI: track 0.00 -> 75.1 mm, vias 0 -> 2
- net SPI1_SCLK: track 0.00 -> 74.2 mm, vias 0 -> 2
- net SPI1_MISO: track 0.00 -> 73.1 mm, vias 0 -> 2
- net UART0_RX: track 0.00 -> 65.1 mm, vias 0 -> 1
- net UART0_TX: track 0.00 -> 63.1 mm, vias 0 -> 1
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- added copper zone on In1.Cu, net RTD2IN-
Other:
- board size 50.8 x 76.2 mm -> 49.5 x 90.8 mm
- net class 5V added: clearance 0.1, trace_width 0.25, via_dia 0.8, via_drill 0.4
- net class 9V added: clearance 0.1, trace_width 0.25, via_dia 0.8, via_drill 0.4
- net class Default: clearance 0.199 -> 0.1; trace_width 0.25 -> 0.2; via_dia 0.8 -> 0.4; via_drill 0.4 -> 0.2
- rule trace_clearance: 0.199 -> 0.1
- rule via_min_drill: 0.3 -> 0.2

Commit message: WIP
Parts:
- added C15: 10 nF, Capacitor_SMD:C_0402_1005Metric, F.Cu at (171.7, 63.2)
- added R17: 4K7, Resistor_SMD:R_0402_1005Metric, F.Cu at (170.9, 65.8)
- added R18: 9K1, Resistor_SMD:R_0603_1608Metric, F.Cu at (170.2, 63.8)
- moved C4 2.35 mm to (168.7, 63.8), turned to 90 degrees
Connections:
- U4 pad 71: +3.3VA -> Net-(R17-Pad2)
Routing:
- net +5V: track 50.2 -> 205.9 mm, vias 0 -> 2
- net +3V3: track 5.18 -> 157.8 mm, vias 0 -> 7
- net Net-(R17-Pad2): track 0.00 -> 101.9 mm, vias 0 -> 2
- net SDC_CLK: track 1.50 -> 69.6 mm, vias 1 -> 3
- net SDC_D0: track 0.00 -> 65.9 mm, vias 0 -> 2
- net SDC_D2: track 0.00 -> 65.1 mm, vias 0 -> 2
- net SDC_D1: track 0.00 -> 64.7 mm, vias 0 -> 2
- net SDC_CMD: track 0.00 -> 62.6 mm, vias 0 -> 2
- net SDC_D3: track 0.00 -> 61.8 mm, vias 0 -> 2
- net +9V: track 29.7 -> 89.9 mm
- net V_SDCARD: track 0.00 -> 57.6 mm, vias 0 -> 2
- net +3.3VA: track 25.4 -> 24.0 mm
- net RTD2IN-: track 136.4 -> 137.7 mm
- net BTN_STEAM: track 50.4 -> 51.5 mm
- net SPI5_MOSI: track 42.4 -> 43.3 mm
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
Commit message: WIP
Parts:
- removed C15: 10 nF, Capacitor_SMD:C_0402_1005Metric
- added NT1: Net-Tie_2, NetTie:NetTie-2_SMD_Pad2.0mm, B.Cu at (160.6, 54.6)
- added R19: R, Resistor_SMD:R_0603_1608Metric, F.Cu at (158.9, 47.2)
- added U7: LM4040DBZ-5, Package_TO_SOT_SMD:SOT-23, F.Cu at (163.1, 47.2)
- J14: moved to B.Cu
- moved J14 51.3 mm to (143.3, 82.5)
- moved J10 6.73 mm to (168.9, 116.3)
- moved R7 6.12 mm to (162.3, 102.6)
- moved R8 6.12 mm to (168.7, 110.2)
- moved R9 6.12 mm to (170.4, 110.2)
- moved U3 6.12 mm to (167.4, 105.4)
- moved R6 6.12 mm to (163.3, 100.6)
- moved U5 5.14 mm to (160.5, 54.6)
- moved C1 4.60 mm to (161.8, 49.8), turned to 180 degrees
- moved C2 3.14 mm to (133.9, 116.1), turned to 0 degrees
- moved C9 3.10 mm to (159.5, 49.8), turned to 0 degrees
- moved J6 2.59 mm to (161.8, 73.7)
- moved J13 2.05 mm to (157.7, 122.2)
- moved U1 2.05 mm to (146.1, 111.5)
- moved J12 1.14 mm to (132.1, 127.0)
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Connections:
- net Net-(R17-Pad2) renamed ADC_VREFP
- net Net-(R4-Pad2) renamed ADC_A0
- C2 pad 2: RTD2IN- -> GND
- C3 pad 2: RTD2IN- -> GND
- C4 pad 2: RTD2IN- -> GND
- C9 pad 1: RTD2IN- -> GND
- D1 pad 1: RTD2IN- -> GND
- D2 pad 1: RTD2IN- -> GND
- D3 pad 1: RTD2IN- -> GND
- J10 pad 2: RTD2IN- -> GND
- J11 pad 2: RTD2IN- -> GND
- J12 pad 2: RTD2IN- -> GND
- J13 pad 6: RTD2IN- -> GND
- J13 pad 9: RTD2IN- -> GND
- J14 pad 3: RTD2IN- -> GND
- J14 pad 5: RTD2IN- -> GND
- J14 pad 9: RTD2IN- -> GND
- J6 pad 1: RTD2IN- -> GND
- J7 pad 3: +5V -> +5VA
- J8 pad 1: RTD2IN- -> GND
- J9 pad 5: RTD2IN- -> GND
- Q1 pad 2: RTD2IN- -> GND
- Q2 pad 2: RTD2IN- -> GND
- Q3 pad 2: RTD2IN- -> GND
- R17 pad 1: +5V -> +5VA
- R6 pad 2: RTD2IN- -> GND
- R8 pad 2: RTD2IN- -> GND
- U1 pad 2: RTD2IN- -> GND
- U2 pad 1: RTD2IN- -> GND
- U3 pad 4: RTD2IN- -> GND
- U4 pad 107: RTD2IN- -> GND
- U4 pad 114: RTD2IN- -> GND
- U4 pad 119: RTD2IN- -> GND
- U4 pad 130: RTD2IN- -> GND
- U4 pad 139: RTD2IN- -> GND
- U4 pad 24: RTD2IN- -> GND
- U4 pad 33: RTD2IN- -> GND
- U4 pad 44: RTD2IN- -> GND
- U4 pad 57: RTD2IN- -> GND
- U4 pad 70: RTD2IN- -> GND
- U5 pad 3: RTD2IN- -> GND
- U5 pad 4: RTD2IN- -> GND
Routing:
- net +5V: track 205.9 -> 0.00 mm, vias 2 -> 0
- net +3V3: track 157.8 -> 0.00 mm, vias 7 -> 0
- net RTD2IN-: track 137.7 -> 0.00 mm, vias 24 -> 0
- net ADC_VREFP: track 101.9 -> 0.00 mm, vias 2 -> 0
- net ADC_A0: track 90.9 -> 0.00 mm, vias 2 -> 0
- net JTAG_RESET: track 90.5 -> 0.00 mm, vias 2 -> 0
- net +9V: track 89.9 -> 0.00 mm
- net JTAG_TDO: track 83.8 -> 0.00 mm, vias 2 -> 0
- net JTAG_TCK: track 83.2 -> 0.00 mm, vias 2 -> 0
- net JTAG_TMS: track 81.0 -> 0.00 mm, vias 2 -> 0
- net ADS1220_DRDY: track 76.3 -> 0.00 mm, vias 2 -> 0
- net ADS1220_CS: track 75.3 -> 0.00 mm, vias 2 -> 0
- net I2C0_SCL: track 75.3 -> 0.00 mm, vias 1 -> 0
- net SPI1_MOSI: track 75.1 -> 0.00 mm, vias 2 -> 0
- net I2C0_SDA: track 75.0 -> 0.00 mm, vias 1 -> 0
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- added copper zone on In1.Cu, net GND
Other:
- board size 49.5 x 90.8 mm -> 49.5 x 119.3 mm

Commit message: WIP
Parts:
- added C15: 10 nF, Capacitor_SMD:C_0402_1005Metric, F.Cu at (159.5, 53.8)
- added C16: 100 nF, Capacitor_SMD:C_0402_1005Metric, F.Cu at (169.2, 58.7)
- added C17: 100 nF, Capacitor_SMD:C_0402_1005Metric, F.Cu at (162.4, 53.8)
- added C18: 100 nF, Capacitor_SMD:C_0402_1005Metric, F.Cu at (169.2, 56.4)
- added C19: 10 nF, Capacitor_SMD:C_0402_1005Metric, F.Cu at (169.2, 61.0)
- added JP1: SolderJumper_2_Open, Jumper:SolderJumper-2_P1.3mm_Open_RoundedPad1.0x1.5mm, B.Cu at (170.2, 46.5)
- added JP2: SolderJumper_2_Open, Jumper:SolderJumper-2_P1.3mm_Open_RoundedPad1.0x1.5mm, B.Cu at (170.3, 50.8)
- added JP3: SolderJumper_2_Open, Jumper:SolderJumper-2_P1.3mm_Open_RoundedPad1.0x1.5mm, B.Cu at (169.8, 42.9)
- added JP4: SolderJumper_2_Open, Jumper:SolderJumper-2_P1.3mm_Open_RoundedPad1.0x1.5mm, B.Cu at (166.9, 60.4)
- added JP5: SolderJumper_2_Open, Jumper:SolderJumper-2_P1.3mm_Open_RoundedPad1.0x1.5mm, B.Cu at (171.2, 60.4)
- added JP6: SolderJumper_2_Open, Jumper:SolderJumper-2_P1.3mm_Open_RoundedPad1.0x1.5mm, B.Cu at (166.1, 56.9)
- added R20: 1K, Resistor_SMD:R_0402_1005Metric, F.Cu at (170.9, 59.9)
- added R21: 680R, Resistor_THT:R_Axial_DIN0204_L3.6mm_D1.6mm_P5.08mm_Horizontal, F.Cu at (166.1, 61.0)
- added R22: 1K, Resistor_SMD:R_0402_1005Metric, F.Cu at (170.9, 57.7)
- added U6: ADS1220xPW, Package_SO:TSSOP-16_4.4x5mm_P0.65mm, F.Cu at (160.8, 58.7)
- J1, J2: footprint Connector_PinHeader_2.54mm:PinHeader_1x02_P2.54mm_Vertical -> Connector_PinHeader_2.54mm:PinHeader_1x04_P2.54mm_Vertical
- J10: footprint Connector_PinHeader_2.54mm:PinHeader_2x05_P2.54mm_Vertical -> Connector_PinHeader_2.54mm:PinHeader_2x05_P2.54mm_Vertical_SMD; moved to B.Cu
- J13: moved to B.Cu
- U1: value 78S04 -> AMS1117-5.0; footprint Package_TO_SOT_THT:TO-220-3_Horizontal_TabDown -> Package_TO_SOT_SMD:SOT-223-3_TabPin2
- moved J8 66.9 mm to (127.0, 76.7)
- moved J9 66.9 mm to (127.0, 62.5)
- moved J10 61.6 mm to (143.0, 60.5)
- moved J6 46.2 mm to (127.3, 42.9)
- moved C2 33.0 mm to (159.3, 95.0)
- moved C3 33.0 mm to (159.3, 92.7)
- moved J13 28.6 mm to (142.7, 97.8), turned to 180 degrees
- moved R8 28.1 mm to (163.8, 82.5)
- moved R9 28.1 mm to (165.6, 82.5)
- moved U3 25.6 mm to (170.7, 80.0), turned to 90 degrees
- moved R19 25.2 mm to (159.8, 72.4)
- moved J12 25.1 mm to (127.3, 102.4)
- moved R6 23.4 mm to (165.0, 77.2)
- moved R7 23.4 mm to (164.1, 79.2)
- moved U7 22.1 mm to (159.8, 69.1)
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Connections:
- net ADS1220_AIN0 renamed ADS1220_1_AIN0
- net ADS1220_AIN1 renamed ADS1220_1_AIN1
- net ADS1220_DRDY renamed ADS1220_1_DRDY
- net ADS1220_REFN0 renamed ADS1220_1_REFN0
- net ADS1220_REFP0 renamed ADS1220_1_REFP0
- C1 pad 1: RTD2IN- -> GNDA
- C10 pad 1: RTD2IN- -> GNDA
- C10 pad 2: ADS1220_AIN2 -> ADS1220_2_AIN0
- C11 pad 1: RTD2IN- -> GNDA
- C12 pad 2: RTD2IN- -> GNDA
- C14 pad 1: RTD2IN- -> GNDA
- C2 pad 1: +9V -> +12V
- C5 pad 1: ADS1220_AIN3 -> ADS1220_2_AIN1
- C5 pad 2: RTD2IN- -> GNDA
- C6 pad 2: RTD2IN- -> GNDA
- C7 pad 1: ADS1220_AIN2 -> ADS1220_2_AIN0
- C7 pad 2: ADS1220_AIN3 -> ADS1220_2_AIN1
- J1 pad 1: ADS1220_IDAC1_RTD1 -> I_IDAC_1_12
- J1 pad 2: ADS1220_IDAC1_RREF -> RTD1IN-
- J11 pad 1: +9V -> +12V
- J12 pad 1: +9V -> +12V
- J2 pad 1: RTD2IN- -> I_IDAC_2_12
- J2 pad 2: ADS1220_IDAC1_RTD1 -> RTD2IN-
- J7 pad 1: RTD2IN- -> GNDA
- NT1 pad 2: RTD2IN- -> GNDA
- R10 pad 1: RTD2IN- -> RTD2IN+
- R10 pad 2: ADS1220_AIN3 -> ADS1220_2_AIN1
- R11 pad 1: ADS1220_IDAC1_RTD1 -> RTD1IN+
- R12 pad 1: ADS1220_IDAC1_RTD1 -> RTD2IN-
- R12 pad 2: ADS1220_AIN2 -> ADS1220_2_AIN0
- R13 pad 1: ADS1220_IDAC1_RREF -> RTD1IN-
- R14 pad 1: ADS1220_IDAC1_RREF -> I_IDAC_1_12
- R15 pad 1: RTD2IN- -> GNDA
- R15 pad 2: ADS1220_IDAC1_RREF -> I_IDAC_1_12
- R16 pad 1: RTD2IN- -> GNDA
- R18 pad 2: RTD2IN- -> GNDA
- R19 pad 1: +9V -> +12V
- R5 pad 2: RTD2IN- -> GNDA
- U1 pad 1: +9V -> GND
- U1 pad 2: GND -> +5V
- U1 pad 3: +5V -> +12V
- U3 pad 8: +9V -> +12V
- U4 pad 36: ADS1220_CS -> Net-(U4-Pad36)
- U4 pad 48: Net-(U4-Pad48) -> ADS1220_1_CS
- U4 pad 72: RTD2IN- -> GNDA
- U4 pad 77: Net-(U4-Pad77) -> ADS1220_2_DRDY
- U4 pad 79: Net-(U4-Pad79) -> ADS1220_2_CS
- U5 pad 2: ADS1220_CS -> ADS1220_1_CS
- U5 pad 5: RTD2IN- -> GNDA
- U5 pad 6: ADS1220_AIN3 -> ADS1220_1_AIN3
- U5 pad 7: ADS1220_AIN2 -> ADS1220_1_AIN2
- U7 pad 2: RTD2IN- -> GNDA
Other:
- board size 49.5 x 119.3 mm -> 54.9 x 66.5 mm
- net class 12V added: clearance 0.127, trace_width 0.254, via_dia 0.6858, via_drill 0.3302
- net class 5V: clearance 0.1 -> 0.127; trace_width 0.25 -> 0.254; via_dia 0.8 -> 0.6858; via_drill 0.4 -> 0.3302
- net class 9V removed
- net class Default: clearance 0.1 -> 0.127; trace_width 0.2 -> 0.254; via_dia 0.4 -> 0.6858; via_drill 0.2 -> 0.3302
- rule trace_clearance: 0.1 -> 0.127
- rule trace_min: 0.2 -> 0.0889
- rule via_min_size: 0.4 -> 0.45
