File: pcb/Silviaduino/Silviaduino.sch (KiCad schematic (older format))
At the start: 45 parts, among them J1 RTD1 Conn, J10 UEXT_Host, J11 ESP8266, J12 Conn_01x02, J2 RTD 2 Conn, J3 SSR1 Conn, J4 SSR2 Conn, J5 SSR3 Conn, J6 PSSR Conn, J7 PXDCR Conn, J8 Btn Conn, J9 Enc Conn, Q1 2N7002, Q2 2N7002, Q3 2N7002, Q4 BSS138, Q5 BSS138, U1 HT7550-1-SOT89, U2 HT7533-1-SOT89, U3 Teensy4.1, U4 PCF8591, U5 MAX31865xAP, U6 MAX31865xAP

Commit message: WIP
Parts:
- removed C5, C6: 10 uF, Capacitor_SMD:C_0402_1005Metric, symbol Device:C_Small
- removed C7, C8: 0.1 uF, Capacitor_SMD:C_0402_1005Metric, symbol Device:C_Small
- removed J11: ESP8266, Connector_PinSocket_2.54mm:PinSocket_2x04_P2.54mm_Vertical, symbol Connector_Generic:Conn_02x04_Odd_Even
- removed J6: PSSR Conn, Connector_PinHeader_2.54mm:PinHeader_1x04_P2.54mm_Vertical, symbol Connector_Generic:Conn_01x04
- removed Q4, Q5: BSS138, Package_TO_SOT_SMD:SOT-23, symbol Transistor_FET:BSS138
- removed R10, R11, R8, R9: 10K, Resistor_SMD:R_0402_1005Metric, symbol Device:R
- removed R4, R5: 10M, Resistor_SMD:R_0402_1005Metric, symbol Device:R
- removed R6, R7: 400R, Resistor_SMD:R_0402_1005Metric, symbol Device:R
- removed U3: Teensy4.1, teensy:Teensy41, symbol teensy:Teensy4.1
- removed U4: PCF8591, Package_SO:SOIC-16W_7.5x10.3mm_P1.27mm, symbol Interface_Expansion:PCF8591
- removed U5, U6: MAX31865xAP, Package_SO:SSOP-20_5.3x7.2mm_P0.65mm, symbol Sensor_Temperature:MAX31865xAP
- added C?: C_Small, symbol Device:C_Small
- added J11: PSSR Conn, symbol Connector_Generic:Conn_01x04
- added J13: Micro_SD_Card, symbol Connector:Micro_SD_Card
- added J6: Display Conn, symbol Connector_Generic:Conn_01x07
- added R4, R7: 5K, symbol Device:R_Small
- added R5, R6: 10K, symbol Device:R_Small
- added TP1, TP2, TP3, TP4, TP5, TP6: TestPoint, symbol Connector:TestPoint
- added U3: MCP6002-xSN, Package_SO:SOIC-8_3.9x4.9mm_P1.27mm, symbol Amplifier_Operational:MCP6002-xSN
- added U4: Portenta_H7, Arduino:Arduino_Portenta_H7, symbol portenta:Portenta_H7
- added U?: ADS1220xPW, Package_SO:TSSOP-16_4.4x5mm_P0.65mm, symbol Analog_ADC:ADS1220xPW
Connections:
- net labels added: ADS1248_CS, ADS1248_DRDY, ADS1248_START, DISPLAY_CS, DISPLAY_DC, DISPLAY_RES, GNDA, I2C0_SCL, I2C0_SDA, MCU_SWCK, MCU_SWDIO, MCU_SWO, PSSR_DAC_3V3, PSSR_DAC_5V, PSSR_EN_3V3, PSSR_EN_9V, PXCDR_AIN, PXDCR_AIN, RTD0_L1, RTD0_L2, RTD0_L3, RTD1_L1, RTD1_L2, RTD1_L3, RTD2_L1, RTD2_L2, RTD2_L3, SDC_CLK, SDC_CMD, SDC_D0, SDC_D1, SDC_D2, SDC_D3, SPI0_MISO, SPI0_MOSI, SPI0_SCLK, SPI1_MISO, SPI1_MOSI, SPI1_SCLK, SPI2_MISO, SPI2_MOSI, SPI2_SCK, SPI5_MISO, SPI5_MOSI, SPI5_SCK, UART0_RX, UART0_TX, UEXT_CS, V_SDCARD
- net labels removed: ESP8266_CHPD, ESP8266_GPIO0, ESP8266_GPIO2, ESP8266_RST, I2C_SCL, I2C_SCL_5V, I2C_SDA, I2C_SDA_5V, PRES_AIN, PROP_SSR_CTRL, PROP_SSR_EN, RX_FROM_ESP8266, TEMP_DRDY0, TEMP_DRDY1, TEMP_DVDD, TEMP_SPI_CS0, TEMP_SPI_CS1, TEMP_SPI_MISO, TEMP_SPI_MOSI, TEMP_SPI_SCK, TEMP_VDD, TX_TO_ESP8266, UEXT_MISO, UEXT_MOSI, UEXT_RXD, UEXT_SCK, UEXT_SCL, UEXT_SDA, UEXT_SSEL, UEXT_TXD
- wire segments 143 -> 63
- no-connect marks 1 -> 60
Other:
- note added: "Connectors"
- note added: "PSSR Op-amp"
- note added: "SPI Mode 1"
- note removed: "I2C Level shifter"
- note removed: "MCU"
- note removed: "Proportional SSR control and Pressure Transducer input"
- note removed: "Teensy"
- moved on the sheet: C9, J1, J10, J12, J2, J3, J4, J5, J7, J8, J9

Commit message: PCB work
Parts:
- removed TP1, TP2, TP3, TP4, TP5, TP6: TestPoint, symbol Connector:TestPoint
- added C10, C11, C12, C14, C5, C6: 10 nF, Capacitor_SMD:C_0402_1005Metric, symbol Device:C_Small
- added C13, C7, C8: 100 nF, Capacitor_SMD:C_0402_1005Metric, symbol Device:C_Small
- added J14: Conn_ARM_JTAG_SWD_10, Connector_PinHeader_1.27mm:PinHeader_2x05_P1.27mm_Vertical_SMD, symbol Connector:Conn_ARM_JTAG_SWD_10
- added R10, R11, R12, R13, R14, R16: 1K, Resistor_SMD:R_0402_1005Metric, symbol Device:R_Small
- added R15: 680R, Resistor_THT:R_Axial_DIN0204_L3.6mm_D1.6mm_P5.08mm_Horizontal, symbol Device:R_Small
- added R8: 3K6, Resistor_SMD:R_0603_1608Metric, symbol Device:R_Small
- added R9: 6K2, Resistor_SMD:R_0603_1608Metric, symbol Device:R_Small
- added unit 2 of U3
- C1: renamed from C?; value C_Small -> 100 nF; footprint (none) -> Capacitor_SMD:C_0402_1005Metric
- C2, C3, C4: footprint Capacitor_SMD:C_0402_1005Metric -> Capacitor_SMD:C_0603_1608Metric
- C9: value 0.1 uF -> 100 nF
- J1, J2: footprint Connector_PinHeader_2.54mm:PinHeader_1x04_P2.54mm_Vertical -> Connector_PinHeader_2.54mm:PinHeader_1x02_P2.54mm_Vertical; symbol Connector:Screw_Terminal_01x04 -> Connector:Screw_Terminal_01x02
- J11: footprint (none) -> Connector_PinHeader_2.54mm:PinHeader_1x04_P2.54mm_Vertical
- J13: footprint (none) -> Connector_Card:microSD_HC_Hirose_DM3AT-SF-PEJM5
- J6: footprint (none) -> Connector_PinHeader_2.54mm:PinHeader_1x07_P2.54mm_Vertical
- R4, R7: value 5K -> 4K7; footprint (none) -> Resistor_SMD:R_0402_1005Metric
- R5, R6: value 10K -> 9K1; footprint (none) -> Resistor_SMD:R_0603_1608Metric
- U1: value HT7550-1-SOT89 -> 78S04; footprint Package_TO_SOT_SMD:SOT-89-3 -> Package_TO_SOT_THT:TO-220-3_Horizontal_TabDown; symbol Regulator_Linear:HT75xx-1-SOT89 -> Regulator_Linear:L7805
- gave numbers to parts that had none: 1
Connections:
- net labels added: ADS1220_AIN0, ADS1220_AIN1, ADS1220_AIN2, ADS1220_AIN3, ADS1220_CS, ADS1220_DRDY, ADS1220_IDAC1_RREF, ADS1220_IDAC1_RTD1, ADS1220_REFN0, ADS1220_REFP0, JTAG_RESET, JTAG_TCK, JTAG_TDO, JTAG_TMS, SPI2_SCLK
- net labels removed: ADS1248_CS, ADS1248_DRDY, ADS1248_START, MCU_SWCK, MCU_SWDIO, MCU_SWO, PXCDR_AIN, RTD0_L1, RTD0_L2, RTD0_L3, RTD1F+, RTD1F-, RTD1_L1, RTD1_L2, RTD1_L3, RTD2F+, RTD2F-, RTD2_L1, RTD2_L2, RTD2_L3, SPI0_MISO, SPI0_MOSI, SPI0_SCLK, SPI2_MISO, SPI2_SCK
- wire segments 63 -> 118
Other:
- note added: "0.515151515 = R7 / R6"
- note added: "1.727272 = R9 / R8"
- note added: "180° C PT100 ~= 168 ohm\n4x gain -> 672 ohm, ~680 ohm"
- note added: "3V3 -> 5V"
- note added: "3V3 -> 9V"
- note added: "5 / 3.3 = 1.5151515"
- note added: "9 / 3.3 = 2.72727272"
- note added: "Non-inverting"
- note added: "Rref = R15"
- note added: "TI ADS1220 datasheet, SBAA235a"
- note added: "https://www.pentronic.se/wp-content/uploads/2019/04/tabell-pt100-2019.pdf"
- note removed: "RTD Power"
- note removed: "https://www.playingwithfusion.com/productview.php?pdid=30"
- moved on the sheet: C1, C9, J10, J11, J6, J8, J9, R6, R7, U3A, U3C, U5

Commit message: WIP
Parts:
- added C15: 10 nF, Capacitor_SMD:C_0402_1005Metric, symbol Device:C_Small
- added R17: 4K7, Resistor_SMD:R_0402_1005Metric, symbol Device:R_Small
- added R18: 9K1, Resistor_SMD:R_0603_1608Metric, symbol Device:R_Small
Connections:
- net +3.3VA: no longer U4.71 (ADC_VREF+)
- net +5V: now also C15.1, R17.1
- net GND: now also C15.2, R18.2
- new net: R17.2, R18.1, U4.71 (ADC_VREF+)
Other:
- moved on the sheet: R4, R5
Changed lines of the file:
@@
 Text GLabel 4200 1300 1    50   Input ~ 0
 SSR3_VNEG
-$Comp
-L power:+5V #PWR011
-U 1 1 60882F52
-P 4550 1300
-F 0 "#PWR011" H 4550 1150 50  0001 C CNN
-F 1 "+5V" H 4565 1473 50  0000 C CNN
-F 2 "" H 4550 1300 50  0001 C CNN
-F 3 "" H 4550 1300 50  0001 C CNN
-	1    4550 1300
-	1    0    0    -1
-$EndComp
 Text GLabel 4650 1300 1    50   Output ~ 0
 PXDCR_AIN
@@
 Text GLabel 10300 4000 2    50   Input ~ 0
 ADS1220_CS
-Text GLabel 11900 9500 0    50   Input ~ 0
+Text GLabel 11600 9800 0    50   Input ~ 0
 PXDCR_AIN
 $Comp
@@
 L Device:R_Small R4
 U 1 1 611CC679
-P 12150 9500
-F 0 "R4" V 12346 9500 50  0000 C CNN
-F 1 "4K7" V 12255 9500 50  0000 C CNN
-F 2 "Resistor_SMD:R_0402_1005Metric" H 12150 9500 50  0001 C CNN
-F 3 "~" H 12150 9500 50  0001 C CNN
-	1    12150 9500
+P 11850 9800
+F 0 "R4" V 12046 9800 50  0000 C CNN
+F 1 "4K7" V 11955 9800 50  0000 C CNN
+F 2 "Resistor_SMD:R_0402_1005Metric" H 11850 9800 50  0001 C CNN
+F 3 "~" H 11850 9800 50  0001 C CNN
+	1    11850 9800
 	0    -1   -1   0
 $EndComp
@@
 L Device:R_Small R5
 U 1 1 611CFFE1
-P 12350 9700
-F 0 "R5" H 12409 9746 50  0000 L CNN
-F 1 "9K1" H 12409 9655 50  0000 L CNN
-F 2 "Resistor_SMD:R_0603_1608Metric" H 12350 9700 50  0001 C CNN
-F 3 "~" H 12350 9700 50  0001 C CNN
-	1    12350 9700
-	1    0    0    -1
-$EndComp
-Wire Wire Line
-	11900 9500 12050 9500
-Wire Wire Line
-	12250 9500 12350 9500
-Wire Wire Line
-	12350 9600 12350 9500
-Connection ~ 12350 9500
-Wire Wire Line
-	12350 9500 13100 9500
+P 12050 10000
+F 0 "R5" H 12109 10046 50  0000 L CNN
+F 1 "9K1" H 12109 9955 50  0000 L CNN
+F 2 "Resistor_SMD:R_0603_1608Metric" H 12050 10000 50  0001 C CNN
+F 3 "~" H 12050 10000 50  0001 C CNN
+	1    12050 10000
+	1    0    0    -1
+$EndComp
+Wire Wire Line
+	11600 9800 11750 9800
+Wire Wire Line
+	11950 9800 12050 9800
+Wire Wire Line
+	12050 9900 12050 9800
 $Comp
 L power:GNDA #PWR0108
 U 1 1 611D5C08
-P 12350 9800
-F 0 "#PWR0108" H 12350 9550 50  0001 C CNN
-F 1 "GNDA" H 12355 9627 50  0000 C CNN
-F 2 "" H 12350 9800 50  0001 C CNN
-F 3 "" H 12350 9800 50  0001 C CNN
-	1    12350 9800
+P 12050 10100
+F 0 "#PWR0108" H 12050 9850 50  0001 C CNN
+F 1 "GNDA" H 12055 9927 50  0000 C CNN
+F 2 "" H 12050 10100 50  0001 C CNN
+F 3 "" H 12050 10100 50  0001 C CNN
+	1    12050 10100
 	1    0    0    -1
 $EndComp
@@
 F 3 "" H 15300 9400 50  0001 C CNN
 	1    15300 9400
-	0    -1   -1   0
-$EndComp
-$Comp
-L power:+3.3VA #PWR0110
-U 1 1 611D9A49
-P 13100 9400
-F 0 "#PWR0110" H 13100 9250 50  0001 C CNN
-F 1 "+3.3VA" V 13115 9527 50  0000 L CNN
-F 2 "" H 13100 9400 50  0001 C CNN
-F 3 "" H 13100 9400 50  0001 C CNN
-	1    13100 9400
 	0    -1   -1   0
 $EndComp
@@
 $EndComp
 $Comp
-L power:+5V #PWR?
+L power:+5V #PWR011
 U 1 1 61AF03EE
 P 1100 7500
-F 0 "#PWR?" H 1100 7350 50  0001 C CNN
+F 0 "#PWR011" H 1100 7350 50  0001 C CNN
 F 1 "+5V" V 1115 7628 50  0000 L CNN
 F 2 "" H 1100 7500 50  0001 C CNN
@@
 	0    -1   -1   0
 $EndComp
+Wire Wire Line
+	12050 9800 12600 9800
+Wire Wire Line
+	12600 9800 12600 9500
+Wire Wire Line
+	12600 9500 13100 9500
+Connection ~ 12050 9800
+$Comp
+L Device:R_Small R17
+U 1 1 619AC9E4
+P 11850 9400
+F 0 "R17" V 12046 9400 50  0000 C CNN
+F 1 "4K7" V 11955 9400 50  0000 C CNN
+F 2 "Resistor_SMD:R_0402_1005Metric" H 11850 9400 50  0001 C CNN
+F 3 "~" H 11850 9400 50  0001 C CNN
+	1    11850 9400
+	0    -1   -1   0
+$EndComp
+$Comp
+L Device:R_Small R18
+U 1 1 619AC9EA
+P 12050 9200
+F 0 "R18" H 11850 9250 50  0000 L CNN
+F 1 "9K1" H 11800 9150 50  0000 L CNN
+F 2 "Resistor_SMD:R_0603_1608Metric" H 12050 9200 50  0001 C CNN
+F 3 "~" H 12050 9200 50  0001 C CNN
+	1    12050 9200
+	-1   0    0    1
+$EndComp
+Wire Wire Line
+	11600 9400 11750 9400
+$Comp
+L power:GNDA #PWR036
+U 1 1 619AC9F3
+P 12050 9100
+F 0 "#PWR036" H 12050 8850 50  0001 C CNN
+F 1 "GNDA" H 12055 8927 50  0000 C CNN
+F 2 "" H 12050 9100 50  0001 C CNN
+F 3 "" H 12050 9100 50  0001 C CNN
+	1    12050 9100
+	-1   0    0    1
+$EndComp
+Wire Wire Line
+	11950 9400 12050 9400
+Wire Wire Line
+	12050 9300 12050 9400
+Connection ~ 12050 9400
+Wire Wire Line
+	12050 9400 13100 9400
+$Comp
+L power:+5VA #PWR033
+U 1 1 619CCBF0
+P 11600 9400
+F 0 "#PWR033" H 11600 9250 50  0001 C CNN
+F 1 "+5VA" V 11615 9527 50  0000 L CNN
+F 2 "" H 11600 9400 50  0001 C CNN
+F 3 "" H 11600 9400 50  0001 C CNN
+	1    11600 9400
+	0    -1   -1   0
+$EndComp
+$Comp
+L power:+5VA #PWR032
+U 1 1 619D1CC0
+P 4550 1300
+F 0 "#PWR032" H 4550 1150 50  0001 C CNN
+F 1 "+5VA" H 4565 1473 50  0000 C CNN
+F 2 "" H 4550 1300 50  0001 C CNN
+F 3 "" H 4550 1300 50  0001 C CNN
+	1    4550 1300
+	1    0    0    -1
+$EndComp
+$Comp
+L power:+5VA #PWR037
+U 1 1 619D41A7
+P 12250 1200
+F 0 "#PWR037" H 12250 1050 50  0001 C CNN
+F 1 "+5VA" V 12265 1328 50  0000 L CNN
+F 2 "" H 12250 1200 50  0001 C CNN
+F 3 "" H 12250 1200 50  0001 C CNN
+	1    12250 1200
+	0    1    1    0
+$EndComp
+$Comp
+L power:+5V #PWR034
+U 1 1 619D5D75
+P 11750 1200
+F 0 "#PWR034" H 11750 1050 50  0001 C CNN
+F 1 "+5V" V 11765 1328 50  0000 L CNN
+F 2 "" H 11750 1200 50  0001 C CNN
+F 3 "" H 11750 1200 50  0001 C CNN
+	1    11750 1200
+	0    -1   -1   0
+$EndComp
+$Comp
+L power:GNDA #PWR035
+U 1 1 619D78A4
+P 12000 1650
+F 0 "#PWR035" H 12000 1400 50  0001 C CNN
+F 1 "GNDA" H 12005 1477 50  0000 C CNN
+F 2 "" H 12000 1650 50  0001 C CNN
+F 3 "" H 12000 1650 50  0001 C CNN
+	1    12000 1650
+	1    0    0    -1
+$EndComp
+$Comp
+L Device:C_Small C15
+U 1 1 619DC825
+P 12000 1400
+F 0 "C15" H 12092 1446 50  0000 L CNN
+F 1 "10 nF" H 12092 1355 50  0000 L CNN
+F 2 "Capacitor_SMD:C_0402_1005Metric" H 12000 1400 50  0001 C CNN
+F 3 "~" H 12000 1400 50  0001 C CNN
+	1    12000 1400
+	1    0    0    -1
+$EndComp
+Wire Wire Line
+	11750 1200 12000 1200
+Wire Wire Line
+	12000 1200 12000 1300
+Connection ~ 12000 1200
+Wire Wire Line
+	12000 1200 12250 1200
+Wire Wire Line
+	12000 1500 12000 1650
 $EndSCHEMATC

Commit message: WIP
Parts:
- removed C15: 10 nF, Capacitor_SMD:C_0402_1005Metric, symbol Device:C_Small
- added NT1: Net-Tie_2, NetTie:NetTie-2_SMD_Pad2.0mm, symbol Device:Net-Tie_2
- added R19: R, Resistor_SMD:R_0603_1608Metric, symbol Device:R
- added U7: LM4040DBZ-5, Package_TO_SOT_SMD:SOT-23, symbol Reference_Voltage:LM4040DBZ-5
Connections:
- net +5V: no longer J7.3 (Pin_3), R17.1
- net +9V: now also R19.1
- net GND: now also NT1.1; no longer C1.1, C10.1, C11.1, C12.2, C14.1, C5.2, C6.2, J2.1 (Pin_1), J7.1 (Pin_1), R10.1, R15.1, R16.1, R18.2, R5.2, U4.72 (ADC_VREF-), U5.5 (AVSS)
- net ADC_VREFP: now reaches R17.2, R18.1, U4.71 (ADC_VREF+)
- net ADC_A0: now reaches R4.2, R5.1, U4.73 (ADC_A0)
- new net +5VA: J7.3 (Pin_3), R17.1, R19.2, U7.1 (K)
- new net GNDA: C1.1, C10.1, C11.1, C12.2, C14.1, C5.2, C6.2, J2.1 (Pin_1), J7.1 (Pin_1), NT1.2, R10.1, R15.1, R16.1, R18.2, R5.2, U4.72 (ADC_VREF-), U5.5 (AVSS), U7.2 (A)
Other:
- moved on the sheet: C4, R17, R18, R4, R5, U2

Commit message: WIP
Parts:
- removed U1: 78S04, Package_TO_SOT_THT:TO-220-3_Horizontal_TabDown, symbol Regulator_Linear:L7805
- added C15, C19: 10 nF, Capacitor_SMD:C_0402_1005Metric, symbol Device:C_Small
- added C16, C17, C18: 100 nF, Capacitor_SMD:C_0402_1005Metric, symbol Device:C_Small
- added JP1, JP2, JP3, JP4, JP5, JP6: SolderJumper_2_Open, Jumper:SolderJumper-2_P1.3mm_Open_RoundedPad1.0x1.5mm, symbol Jumper:SolderJumper_2_Open
- added R20, R22: 1K, Resistor_SMD:R_0402_1005Metric, symbol Device:R_Small
- added R21: 680R, Resistor_THT:R_Axial_DIN0204_L3.6mm_D1.6mm_P5.08mm_Horizontal, symbol Device:R_Small
- added U1: AMS1117-5.0, Package_TO_SOT_SMD:SOT-223-3_TabPin2, symbol Regulator_Linear:AMS1117-5.0
- added U6: ADS1220xPW, Package_SO:TSSOP-16_4.4x5mm_P0.65mm, symbol Analog_ADC:ADS1220xPW
- J1, J2: footprint Connector_PinHeader_2.54mm:PinHeader_1x02_P2.54mm_Vertical -> Connector_PinHeader_2.54mm:PinHeader_1x04_P2.54mm_Vertical; symbol Connector:Screw_Terminal_01x02 -> Connector:Screw_Terminal_01x04
- J10: footprint Connector_PinHeader_2.54mm:PinHeader_2x05_P2.54mm_Vertical -> Connector_PinHeader_2.54mm:PinHeader_2x05_P2.54mm_Vertical_SMD
Connections:
- net +3.3VA: now also C18.2, U6.12 (AVDD)
- net +3V3: now also C16.2, U6.13 (DVDD)
- net +5V: now also U1.2 (VO)
- net GND: now also C16.1, U1.1 (GND), U6.3 (CLK), U6.4 (DGND)
- net GNDA: now also C15.2, C18.1, C19.1, R21.1, R22.1, U6.5 (AVSS); no longer J2.1 (Pin_1), R10.1
- net SPI1_MISO: now also U6.16 (DIN)
- net SPI1_MOSI: now also U6.15 (DOUT/~DRDY)
- net SPI1_SCLK: now also U6.1 (SCLK)
- net ADS1220_1_CS: now reaches U4.48 (GPIO_1)
- net ADS1220_1_CS: now also U5.2 (~CS)
- net ADS1220_2_DRDY: now reaches U4.77 (ADC_A2)
- net ADS1220_2_DRDY: now also U6.14 (~DRDY)
- net ADS1220_2_CS: now reaches U4.79 (ADC_A3)
- net ADS1220_2_CS: now also U6.2 (~CS)
- net +9V renamed +12V
- net +12V: now also U1.3 (VI)
- net ADS1220_AIN0 renamed ADS1220_1_AIN0
- net ADS1220_AIN1 renamed ADS1220_1_AIN1
- net ADS1220_AIN2 renamed ADS1220_2_AIN0
- net ADS1220_2_AIN0: now also U6.11 (AIN0/REFP1); no longer U5.7 (AIN2)
- net ADS1220_AIN3 renamed ADS1220_2_AIN1
- net ADS1220_2_AIN1: now also U6.10 (AIN1); no longer U5.6 (AIN3/REFN1)
- net ADS1220_CS: no longer names the net of U4.36 (SPI1_CS)
- net ADS1220_CS: no longer U5.2 (~CS)
- net ADS1220_DRDY renamed ADS1220_1_DRDY
- net ADS1220_IDAC1_RREF renamed I_IDAC_1_12
- net I_IDAC_1_12: now also J1.1 (Pin_1), JP2.1 (A); no longer J1.2 (Pin_2), R13.1
- net ADS1220_IDAC1_RTD1 renamed RTD2IN-
- net RTD2IN-: now also JP5.2 (B), JP6.2 (B); no longer J1.1 (Pin_1), R11.1
- net ADS1220_REFN0 renamed ADS1220_1_REFN0
- net ADS1220_REFP0 renamed ADS1220_1_REFP0
- new net ADS1220_1_AIN2: JP3.1 (A), U5.7 (AIN2)
- new net ADS1220_1_AIN3: J1.4 (Pin_4), J2.4 (Pin_4), JP1.2 (B), U5.6 (AIN3/REFN1)
- new net ADS1220_2_AIN2: JP6.1 (A), U6.7 (AIN2)
- new net ADS1220_2_AIN3: JP4.2 (B), U6.6 (AIN3/REFN1)
- new net ADS1220_2_REFN0: C17.1, C19.2, R22.2, U6.8 (REFN0)
- new net ADS1220_2_REFP0: C15.1, C17.2, R20.2, U6.9 (REFP0)
- new net I_IDAC_2_12: J2.1 (Pin_1), JP5.1 (A), R20.1, R21.2
- new net RTD1IN+: J1.3 (Pin_3), JP1.1 (A), R11.1
- new net RTD1IN-: J1.2 (Pin_2), JP2.2 (B), JP3.2 (B), R13.1
- new net RTD2IN+: J2.3 (Pin_3), JP4.1 (A), R10.1
- no-connect marks 60 -> 58
Other:
- moved on the sheet: C1, C12, C13, C14, C9, NT1, R14, R15, R16, R17, R18, R19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
